File: hardware/0v2/dd8_0v2/dd8_0v2.kicad_sch (KiCad schematic)
At the start: 13 parts, among them J1 Conn_Coaxial, J2 Banana socket, SW1 SW_Push, U1 W65C51NxP, U2 W65C02SxP, U3 AS7C256B, U4 AT28C64B, U5 chip_selector, Y1 1.8432MHz

Commit message: updates
Parts:
- removed U5: chip_selector, symbol dd8_components_library:ics_0v2
- added U6: ~, symbol dd8_components_library:ics_0v2
Connections:
- net +5V: now also U6. (VSS)
- net GND: now also U6. (VSS)
- net a13: now also U6.4 (A13)
- net a14: now also U6.5 (A14)
- net a15: now also U6.6 (A15)
- net ce1_uart: now also U6.16 (CE1_{UART})
- net clk: now also U6.2 (CLK)
- net r~{w}: now also U6.1 (R~{W})
- net ~{ce2_uart}: now also U6.17 (~{CE2_{UART}})
- net ~{ce_ram}: now also U6.12 (~{CE_{RAM}})
- net ~{ce_rom}: now also U6.11 (~{CE_{ROM}})
- net ~{oe}: now also U6.9 (~{OE})
- net ~{we}: now also U6.8 (~{WE})

Commit message: A lot of updates
Parts:
- removed U6: ~, symbol dd8_components_library:ics_0v2
- added C11, C3, C4, C5, C6, C7, C8: 100n, Capacitor_THT:C_Disc_D3.0mm_W1.6mm_P2.50mm, symbol Device:C
- added C12, C2: 10uF, Capacitor_THT:CP_Radial_D5.0mm_P2.50mm, symbol Device:C_Polarized
- added D1: LED, LED_THT:LED_D3.0mm, symbol Device:LED
- added D2: D_Schottky, Diode_THT:D_DO-35_SOD27_P7.62mm_Horizontal, symbol Device:D_Schottky
- added J3: Conn_02x27_Odd_Even, Connector_PinSocket_2.54mm:PinSocket_2x27_P2.54mm_Vertical, symbol Connector_Generic:Conn_02x27_Odd_Even
- added J4: Conn_01x14, Connector_PinHeader_2.54mm:PinHeader_2x07_P2.54mm_Vertical, symbol Connector_Generic:Conn_01x14
- added J5, J6: Conn_01x02_Pin, Connector_PinSocket_2.54mm:PinSocket_1x02_P2.54mm_Vertical, symbol Connector:Conn_01x02_Pin
- added JP1, JP2, JP3, JP4, JP5: Jumper_2_Open, Jumper:SolderJumper-2_P1.3mm_Open_Pad1.0x1.5mm, symbol Jumper:Jumper_2_Open
- added JP6, JP7, JP8: Jumper_2_Bridged, Connector_PinHeader_2.54mm:PinHeader_1x02_P2.54mm_Vertical, symbol Jumper:Jumper_2_Bridged
- added R4: 1k, Resistor_THT:R_Axial_DIN0204_L3.6mm_D1.6mm_P2.54mm_Vertical, symbol Device:R
- added U5: ~, Package_LCC:PLCC-44_THT-Socket, symbol dd8_components_library:ics_0v2
- C1: footprint (none) -> Capacitor_THT:C_Disc_D3.0mm_W1.6mm_P2.50mm
- J1: footprint (none) -> Connector_Coaxial:BNC_Amphenol_B6252HB-NPP3G-50_Horizontal
- J2: footprint (none) -> dd8_footprints_library:Bannana_Jack_2Pin
- R1, R2: footprint (none) -> Resistor_THT:R_Axial_DIN0204_L3.6mm_D1.6mm_P2.54mm_Vertical
- R3: footprint (none) -> Resistor_THT:R_Axial_DIN0204_L3.6mm_D1.6mm_P5.08mm_Horizontal
- SW1: footprint (none) -> Button_Switch_THT:SW_PUSH_6mm_H5mm
- U3: footprint (none) -> Package_DIP:DIP-28_W7.62mm
- U4: footprint (none) -> Socket:DIP_Socket-28_W11.9_W12.7_W15.24_W17.78_W18.5_3M_228-1277-00-0602J
- Y1: footprint (none) -> Crystal:Crystal_HC18-U_Vertical
Connections:
- net ce1_uart is gone; now on net VCC: U1.2 (CS1)
- net GND: now also C11.2, C12.2, C2.2, C3.2, C4.2, C5.2, C6.2, C7.2, C8.2, D1.1 (K), J3.14 (Pin_14), J3.15 (Pin_15), J3.18 (Pin_18), J3.2 (Pin_2), J3.20 (Pin_20), J3.26 (Pin_26), J3.32 (Pin_32), J3.38 (Pin_38), J3.44 (Pin_44), J3.50 (Pin_50), J3.8 (Pin_8), J4.2 (Pin_2), J5.2 (Pin_2), J6.2 (Pin_2), U5.10 (VSS_0), U5.22 (VSS_1), U5.30 (VSS_2), U5.42 (VSS_3)
- net a0: now also J3.33 (Pin_33), U5.20 (A0)
- net a1: now also J3.34 (Pin_34), U5.24 (A1)
- net a10: now also J3.47 (Pin_47), U5.39 (A10)
- net a11: now also J3.48 (Pin_48), U5.40 (A11)
- net a12: now also J3.51 (Pin_51), U5.41 (A12)
- net a13: now also J3.52 (Pin_52), U5.37 (A13)
- net a14: now also J3.53 (Pin_53), U5.33 (A14)
- net a15: now also J3.54 (Pin_54), U5.31 (A15)
- net a2: now also J3.35 (Pin_35), U5.21 (A2)
- net a3: now also J3.36 (Pin_36), U5.26 (A3)
- net a4: now also J3.39 (Pin_39), U5.25 (A4)
- net a5: now also J3.40 (Pin_40), U5.27 (A5)
- net a6: now also J3.41 (Pin_41), U5.28 (A6)
- net a7: now also J3.42 (Pin_42), U5.29 (A7)
- net a8: now also J3.45 (Pin_45), U5.34 (A8)
- net a9: now also J3.46 (Pin_46), U5.36 (A9)
- net clk: now also J6.1 (Pin_1), U5.43 (CLK); no longer U1.27 (ϕ2), U2.37 (ϕ0)
- net d0: now also J3.21 (Pin_21)
- net d1: now also J3.22 (Pin_22)
- net d2: now also J3.23 (Pin_23)
- net d3: now also J3.24 (Pin_24)
- net d4: now also J3.27 (Pin_27)
- net d5: now also J3.28 (Pin_28)
- net d6: now also J3.29 (Pin_29)
- net d7: now also J3.30 (Pin_30)
- net reset: now also C11.1, C2.1, J3.1 (Pin_1)
- net r~{w}: now also J3.4 (Pin_4), U5.19 (R~{W})
- net ~{ce_ram}: now also U5.8 (~{CE_{RAM}}); no longer U4.20 (~{CE})
- net ~{ce_rom}: now also U4.20 (~{CE}), U5.6 (~{CE_{ROM}})
- net ~{irq}: now also D2.2 (A), J3.5 (Pin_5); no longer U1.26 (~{IRQ})
- net ~{oe}: now also J3.6 (Pin_6), U5.5 (~{OE})
- net ~{we}: now also J3.7 (Pin_7), U5.4 (~{WE}); no longer U4.27 (~{WE})
- net txd: now reaches U1.10 (TxD)
- net txd: now also J4.4 (Pin_4)
- net ~{dts}: now reaches U1.11 (~{DTR})
- net ~{dts}: now also JP3.1 (A)
- net rxd: now reaches U1.12 (RxD)
- net rxd: now also J4.5 (Pin_5)
- net ~{dcd}: now reaches U1.16 (~{DCD})
- net ~{dcd}: now also JP5.1 (A)
- net ~{dsr}: now reaches U1.17 (~{DSR})
- net ~{dsr}: now also JP4.1 (A)
- net ~{rts}: now reaches U1.8 (~{RTS})
- net ~{rts}: now also JP2.1 (A)
- net ~{cts}: now reaches U1.9 (~{CTS})
- net ~{cts}: now also JP1.1 (A)
- net +5V renamed VCC
- net VCC: now also U4.27 (~{WE}), C12.1, C3.1, C4.1, C5.1, C6.1, C7.1, C8.1, J3.19 (Pin_19), J3.25 (Pin_25), J3.3 (Pin_3), J3.31 (Pin_31), J3.37 (Pin_37), J3.43 (Pin_43), J3.49 (Pin_49), J3.9 (Pin_9), J4.1 (Pin_1), J4.3 (Pin_3), J5.1 (Pin_1), JP6.1 (A), JP7.1 (A), JP8.1 (A), R4.2, U5.15 (VCC_1), U5.23 (VCC_2), U5.3 (VCC_0), U5.35 (VCC_3); no longer U2.36 (BE), U2.38 (~{SO}), U2.6 (~{NMI})
- net ~{ce2_uart} renamed ~{ce_uart}
- net ~{ce_uart}: now also U5.9 (~{CE_{UART}})
- new net: J4.10 (Pin_10), JP5.2 (B)
- new net: J4.6 (Pin_6), JP1.2 (B)
- new net: J4.7 (Pin_7), JP2.2 (B)
- new net: J4.8 (Pin_8), JP3.2 (B)
- new net: J4.9 (Pin_9), JP4.2 (B)
- new net: JP8.2 (B), U2.6 (~{NMI})
- new net: JP7.2 (B), U2.36 (BE)
- new net: D2.1 (K), U1.26 (~{IRQ})
- new net: JP6.2 (B), U2.38 (~{SO})
- new net: D1.2 (A), R4.1
- new net clk2: J3.16 (Pin_16), U1.27 (ϕ2), U2.37 (ϕ0), U5.12 (R5)
- new net clk_aux: J3.17 (Pin_17), U5.14 (R4)
- new net res_0: J3.11 (Pin_11), U5.17 (R0)
- new net res_1: J3.13 (Pin_13), U5.18 (R1)
- new net res_2: J3.10 (Pin_10), U5.11 (R2)
- new net res_3: J3.12 (Pin_12), U5.16 (R3)
Other:
- note added: "dd8 0v2 - prototype board"
- note removed: "0000-7FFF"
- note removed: "32k SRAM"
- note removed: "8k ROM"
- note removed: "ADDR RANGE"
- note removed: "C000-C003"
- note removed: "DEVICE"
- note removed: "E000-FFFF"
- note removed: "UART"
- note removed: "dd8 0v2 - multi processor 8 bit computer"
- moved on the sheet: C1, J2, R1, R2, R3, SW1, U1, U2, U3, U4, Y1
