File: tools/hardware/EPMDevBoard/EpmDevBoard/EpmDevBoard.kicad_sch (KiCad schematic)
At the start: 7 parts, among them J1 Conn_01x22_Pin, J2 Conn_01x22_Pin, J5 Conn_01x22_Pin, J6 Conn_01x22_Pin

Commit message: Major graphics card update
Parts:
- removed J1, J2, J5, J6: Conn_01x22_Pin, Connector_PinHeader_2.54mm:PinHeader_1x22_P2.54mm_Vertical, symbol Connector:Conn_01x22_Pin
- removed U3: ~, Package_LCC:PLCC-44_THT-Socket, symbol dd8_components_library:EPM7064_44
- removed U5: ~, Package_LCC:PLCC-84_THT-Socket, symbol dd8_components_library:EPM7128_84
- added C1, C10, C11, C2, C3, C4, C5, C6, C7, C8, C9: 100n, Capacitor_THT:C_Disc_D3.0mm_W1.6mm_P2.50mm, symbol Device:C
- added J1, J15, J17, J18, J19, J2, J3, J4: Conn_01x11_Pin, Connector_PinHeader_2.54mm:PinHeader_1x11_P2.54mm_Vertical, symbol Connector:Conn_01x11_Pin
- added J10, J11, J12, J5, J6, J7, J8, J9: Conn_01x21_Pin, Connector_PinSocket_2.54mm:PinSocket_1x21_P2.54mm_Vertical, symbol Connector:Conn_01x21_Pin
- added J13, J14: Conn_02x05_Odd_Even, Connector_IDC:IDC-Header_2x05_P2.54mm_Vertical, symbol Connector_Generic:Conn_02x05_Odd_Even
- added J20: Conn_Coaxial, Connector_Coaxial:BNC_Amphenol_B6252HB-NPP3G-50_Horizontal, symbol Connector:Conn_Coaxial
- added J21: Conn_02x06_Odd_Even, Connector_PinHeader_2.54mm:PinHeader_2x06_P2.54mm_Vertical, symbol Connector_Generic:Conn_02x06_Odd_Even
- added JP1: Jumper_1_Open, Connector_PinHeader_2.54mm:PinHeader_2x01_P2.54mm_Vertical, symbol Jumper:Jumper_2_Open
- added JP2: Jumper_2_Open, Connector_PinHeader_2.54mm:PinHeader_2x01_P2.54mm_Vertical, symbol Jumper:Jumper_2_Open
- added JP3: Jumper_3_Open, Jumper:SolderJumper-2_P1.3mm_Open_Pad1.0x1.5mm, symbol Jumper:Jumper_2_Open
- added JP4: Jumper_4_Open, Jumper:SolderJumper-2_P1.3mm_Open_Pad1.0x1.5mm, symbol Jumper:Jumper_2_Open
- added R1, R2, R3, R4, R5, R6, R7, R8: 10K, Resistor_THT:R_Axial_DIN0204_L3.6mm_D1.6mm_P5.08mm_Horizontal, symbol Device:R
- added U3: EPM7128S, Package_LCC:PLCC-84_THT-Socket, symbol dd8_components_library:EPM7128_84
- U1: value ~ -> EPM7064S
Connections:
- net VCC_2: now reaches U1.23 (VCC)
- net VCC_2: now also U1.15 (VCC), U1.3 (VCC), U1.35 (VCC), C1.1, C2.1, C3.1, C4.1, J1.4 (Pin_4), J14.4 (Pin_4), J15.4 (Pin_4), J17.6 (Pin_6), J18.7 (Pin_7), J19.9 (Pin_9), J2.9 (Pin_9), J3.7 (Pin_7), J4.6 (Pin_6), JP1.2 (B), R6.1, R7.1, R8.1
- net TCLK_2: now reaches U1.32 (I/O_(TCK))
- net TCLK_2: now also J14.1 (Pin_1), J18.4 (Pin_4), J3.4 (Pin_4), R5.2
- net at U1.33 (I/O): now also J18.5 (Pin_5), J3.5 (Pin_5)
- net at U1.34 (I/O): now also J18.6 (Pin_6), J3.6 (Pin_6)
- net at U1.36 (I/O): now also J18.8 (Pin_8), J3.8 (Pin_8)
- net at U1.37 (I/O): now also J18.9 (Pin_9), J3.9 (Pin_9)
- net TDO_2: now reaches U1.38 (I/O_(TDO))
- net TDO_2: now also J14.3 (Pin_3), J18.10 (Pin_10), J3.10 (Pin_10), R6.2
- net at U1.39 (I/O): now also J18.11 (Pin_11), J3.11 (Pin_11)
- net at U1.40 (I/O): now also J1.11 (Pin_11), J15.11 (Pin_11)
- net at U1.41 (I/O): now also J1.10 (Pin_10), J15.10 (Pin_10)
- net at U1.24 (I/O): now also J17.7 (Pin_7), J4.7 (Pin_7)
- net GND: now reaches U1.42 (GND)
- net GND: now also U1.10 (GND), U1.22 (GND), U1.30 (GND), C1.2, C10.2, C11.2, C2.2, C3.2, C4.2, C5.2, C6.2, C7.2, C8.2, C9.2, J1.9 (Pin_9), J10.21 (Pin_21), J10.8 (Pin_8), J11.6 (Pin_6), J12.10 (Pin_10), J12.15 (Pin_15), J13.10 (Pin_10), J13.2 (Pin_2), J14.10 (Pin_10), J14.2 (Pin_2), J15.9 (Pin_9), J17.5 (Pin_5), J18.2 (Pin_2), J19.4 (Pin_4), J2.4 (Pin_4), J20.2 (Ext), J21.1 (Pin_1), J21.11 (Pin_11), J21.3 (Pin_3), J21.5 (Pin_5), J21.7 (Pin_7), J21.9 (Pin_9), J3.2 (Pin_2), J4.5 (Pin_5), J5.6 (Pin_6), J6.10 (Pin_10), J6.15 (Pin_15), J7.21 (Pin_21), J7.8 (Pin_8), J8.14 (Pin_14), J8.5 (Pin_5), J9.14 (Pin_14), J9.5 (Pin_5), R1.1, R5.1, U3.19 (GDN), U3.32 (GND), U3.42 (GND), U3.47 (GND), U3.59 (GND), U3.7 (GND), U3.82 (GND)
- net CLK_2: now reaches U1.43 (IN/GCLK1)
- net CLK_2: now also J1.8 (Pin_8), J15.8 (Pin_8), JP3.1 (A)
- net at U1.44 (IN/OE1): now also J1.7 (Pin_7), J15.7 (Pin_7)
- net at U1.25 (I/O): now also J17.8 (Pin_8), J4.8 (Pin_8)
- net at U1.26 (I/O): now also J17.9 (Pin_9), J4.9 (Pin_9)
- net at U1.27 (I/O): now also J17.10 (Pin_10), J4.10 (Pin_10)
- net at U1.28 (I/O): now also J17.11 (Pin_11), J4.11 (Pin_11)
- net at U1.29 (I/O): now also J18.1 (Pin_1), J3.1 (Pin_1)
- net at U1.31 (I/O): now also J18.3 (Pin_3), J3.3 (Pin_3)
- net at U1.1 (IN/GCLRn): now also J1.6 (Pin_6), J15.6 (Pin_6)
- net at U1.11 (I/O): now also J19.5 (Pin_5), J2.5 (Pin_5)
- net at U1.12 (I/O): now also J19.6 (Pin_6), J2.6 (Pin_6)
- net TMS_2: now reaches U1.13 (I/O(TMS))
- net TMS_2: now also J14.5 (Pin_5), J19.7 (Pin_7), J2.7 (Pin_7), R7.2
- net at U1.14 (I/O): now also J19.8 (Pin_8), J2.8 (Pin_8)
- net at U1.16 (I/O): now also J19.10 (Pin_10), J2.10 (Pin_10)
- net at U1.17 (I/O): now also J19.11 (Pin_11), J2.11 (Pin_11)
- net at U1.18 (I/O): now also J17.1 (Pin_1), J4.1 (Pin_1)
- net at U1.19 (I/O): now also J17.2 (Pin_2), J4.2 (Pin_2)
- net at U1.2 (IN/OE2/GCLK2): now also J1.5 (Pin_5), J15.5 (Pin_5)
- net at U1.20 (I/O): now also J17.3 (Pin_3), J4.3 (Pin_3)
- net at U1.21 (I/O): now also J17.4 (Pin_4), J4.4 (Pin_4)
- net at U1.4 (I/O): now also J1.3 (Pin_3), J15.3 (Pin_3)
- net at U1.5 (I/O): now also J1.2 (Pin_2), J15.2 (Pin_2)
- net at U1.6 (I/O): now also J1.1 (Pin_1), J15.1 (Pin_1)
- net TDI_2: now reaches U1.7 (I/O(TDI))
- net TDI_2: now also J14.9 (Pin_9), J19.1 (Pin_1), J2.1 (Pin_1), R8.2
- net at U1.8 (I/O): now also J19.2 (Pin_2), J2.2 (Pin_2)
- net at U1.9 (I/O): now also J19.3 (Pin_3), J2.3 (Pin_3)
- new net: J10.1 (Pin_1), J7.1 (Pin_1), U3.12 (I/O)
- new net: J10.10 (Pin_10), J7.10 (Pin_10), U3.21 (I/O)
- new net: J10.11 (Pin_11), J7.11 (Pin_11), U3.22 (I/O)
- new net: J10.13 (Pin_13), J7.13 (Pin_13), U3.24 (I/O)
- new net: J10.14 (Pin_14), J7.14 (Pin_14), U3.25 (I/O)
- new net: J10.16 (Pin_16), J7.16 (Pin_16), U3.27 (I/O)
- new net: J10.17 (Pin_17), J7.17 (Pin_17), U3.28 (I/O)
- new net: J10.18 (Pin_18), J7.18 (Pin_18), U3.29 (I/O)
- new net: J10.19 (Pin_19), J7.19 (Pin_19), U3.30 (I/O)
- new net: J10.20 (Pin_20), J7.20 (Pin_20), U3.31 (I/O)
- new net: J10.4 (Pin_4), J7.4 (Pin_4), U3.15 (I/O)
- new net: J10.5 (Pin_5), J7.5 (Pin_5), U3.16 (I/O)
- new net: J10.6 (Pin_6), J7.6 (Pin_6), U3.17 (I/O)
- new net: J10.7 (Pin_7), J7.7 (Pin_7), U3.18 (I/O)
- new net: J10.9 (Pin_9), J7.9 (Pin_9), U3.20 (I/O)
- new net: J8.1 (Pin_1), J9.1 (Pin_1), U3.11 (I/O)
- new net: J8.10 (Pin_10), J9.10 (Pin_10), U3.2 (IN/OE2/GCLK2)
- new net: J8.11 (Pin_11), J9.11 (Pin_11), U3.1 (IN/GLCRn)
- new net: J8.12 (Pin_12), J9.12 (Pin_12), U3.84 (IN/OE1)
- new net: J8.15 (Pin_15), J9.15 (Pin_15), U3.81 (I/O)
- new net: J8.16 (Pin_16), J9.16 (Pin_16), U3.80 (I/O)
- new net: J8.17 (Pin_17), J9.17 (Pin_17), U3.79 (I/O)
- new net: J8.19 (Pin_19), J9.19 (Pin_19), U3.77 (I/O)
- new net: J8.2 (Pin_2), J9.2 (Pin_2), U3.10 (I/O)
- new net: J8.20 (Pin_20), J9.20 (Pin_20), U3.76 (I/O)
- new net: J8.21 (Pin_21), J9.21 (Pin_21), U3.75 (I/O)
- new net: J8.3 (Pin_3), J9.3 (Pin_3), U3.9 (I/O)
- new net: J8.4 (Pin_4), J9.4 (Pin_4), U3.8 (I/O)
- new net: J8.6 (Pin_6), J9.6 (Pin_6), U3.6 (I/O)
- new net: J8.7 (Pin_7), J9.7 (Pin_7), U3.5 (I/O)
- new net: J8.8 (Pin_8), J9.8 (Pin_8), U3.4 (I/O)
- new net: J21.10 (Pin_10), J21.12 (Pin_12), J21.2 (Pin_2), J21.4 (Pin_4), J21.6 (Pin_6), J21.8 (Pin_8), JP1.1 (A), JP2.1 (A)
- new net: J12.1 (Pin_1), J6.1 (Pin_1), U3.33 (I/O)
- new net: J12.2 (Pin_2), J6.2 (Pin_2), U3.34 (I/O)
- new net: J12.3 (Pin_3), J6.3 (Pin_3), U3.35 (I/O)
- new net: J12.4 (Pin_4), J6.4 (Pin_4), U3.36 (I/O)
- new net: J12.5 (Pin_5), J6.5 (Pin_5), U3.37 (I/O)
- new net: J12.7 (Pin_7), J6.7 (Pin_7), U3.39 (I/O)
- new net: J12.8 (Pin_8), J6.8 (Pin_8), U3.40 (I/O)
- new net: J12.9 (Pin_9), J6.9 (Pin_9), U3.41 (I/O)
- new net: J12.12 (Pin_12), J6.12 (Pin_12), U3.44 (I/O)
- new net: J12.13 (Pin_13), J6.13 (Pin_13), U3.45 (I/O)
- new net: J12.14 (Pin_14), J6.14 (Pin_14), U3.46 (I/O)
- new net: J12.16 (Pin_16), J6.16 (Pin_16), U3.48 (I/O)
- new net: J12.17 (Pin_17), J6.17 (Pin_17), U3.49 (I/O)
- new net: J12.18 (Pin_18), J6.18 (Pin_18), U3.50 (I/O)
- new net: J12.19 (Pin_19), J6.19 (Pin_19), U3.51 (I/O)
- new net: J12.20 (Pin_20), J6.20 (Pin_20), U3.52 (I/O)
- new net: J11.1 (Pin_1), J5.1 (Pin_1), U3.54 (I/O)
- new net: J11.2 (Pin_2), J5.2 (Pin_2), U3.55 (I/O)
- new net: J11.3 (Pin_3), J5.3 (Pin_3), U3.56 (I/O)
- new net: J11.4 (Pin_4), J5.4 (Pin_4), U3.57 (I/O)
- new net: J11.5 (Pin_5), J5.5 (Pin_5), U3.58 (I/O)
- new net: J11.7 (Pin_7), J5.7 (Pin_7), U3.60 (I/O)
- new net: J11.8 (Pin_8), J5.8 (Pin_8), U3.61 (I/O)
- new net: J11.10 (Pin_10), J5.10 (Pin_10), U3.63 (I/O)
- new net: J11.11 (Pin_11), J5.11 (Pin_11), U3.64 (I/O)
- new net: J11.12 (Pin_12), J5.12 (Pin_12), U3.65 (I/O)
- new net: J11.14 (Pin_14), J5.14 (Pin_14), U3.67 (I/O)
- new net: J11.15 (Pin_15), J5.15 (Pin_15), U3.68 (I/O)
- new net: J11.16 (Pin_16), J5.16 (Pin_16), U3.69 (I/O)
- new net: J11.17 (Pin_17), J5.17 (Pin_17), U3.70 (I/O)
- new net: J11.19 (Pin_19), J5.19 (Pin_19), U3.72 (I/O)
- new net: J11.20 (Pin_20), J5.20 (Pin_20), U3.73 (I/O)
- new net: J11.21 (Pin_21), J5.21 (Pin_21), U3.74 (I/O)
- new net: J20.1 (In), JP3.2 (B), JP4.2 (B)
- new net CLK_1: J8.13 (Pin_13), J9.13 (Pin_13), JP4.1 (A), U3.83 (IN/GCLK1)
- new net TCLK_1: J11.9 (Pin_9), J13.1 (Pin_1), J5.9 (Pin_9), R1.2, U3.62 (I/O(TCK))
- new net TDI_1: J10.3 (Pin_3), J13.9 (Pin_9), J7.3 (Pin_3), R4.2, U3.14 (I/O(TDI))
- new net TDO_1: J11.18 (Pin_18), J13.3 (Pin_3), J5.18 (Pin_18), R2.2, U3.71 ((TDO))
- new net TMS_1: J10.12 (Pin_12), J13.5 (Pin_5), J7.12 (Pin_12), R3.2, U3.23 (I/O(TMS))
- new net VCC_1: C10.1, C11.1, C5.1, C6.1, C7.1, C8.1, C9.1, J10.15 (Pin_15), J10.2 (Pin_2), J11.13 (Pin_13), J12.11 (Pin_11), J12.21 (Pin_21), J12.6 (Pin_6), J13.4 (Pin_4), J5.13 (Pin_13), J6.11 (Pin_11), J6.21 (Pin_21), J6.6 (Pin_6), J7.15 (Pin_15), J7.2 (Pin_2), J8.18 (Pin_18), J8.9 (Pin_9), J9.18 (Pin_18), J9.9 (Pin_9), JP2.2 (B), R2.1, R3.1, R4.1, U3.13 (VCCIO), U3.26 (VCCIO), U3.3 (VCCINT), U3.38 (VCCIO), U3.43 (VCCINT), U3.53 (VCCIO), U3.66 (VCCIO), U3.78 (VCCIO)
Other:
- note added: "100n"
