File: hardware/kicad/dd8_computer/dd8_computer.kicad_sch (KiCad schematic)
At the start: 0 parts

Commit message: update
Other:
- sheet vga_module renamed gfx_module
- sheet gfx_module: file vga_module.kicad_sch -> gfx_module.kicad_sch
- sheet gfx_module ports: added addr_{cpu}[0..15], clk_{2}, data_{cpu}[0..7], gfx_{dma_act}, gfx_{fr_end}, gfx_{fr_prog}, gfx_{fr_start}, ~{gfx_{ce}}, ~{oe_{cpu}}, ~{plt_{cs}}, ~{ramb0_{ce}}, ~{we_{cpu}}; removed none
Changed lines of the file:
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@@
 			(color 0 0 0 0.0000)
 		)
-		(property "Sheetname" "vga_module"
+		(property "Sheetname" "gfx_module"
 			(at 190.5 121.4624 0)
 			(effects
@@
 			)
 		)
-		(property "Sheetfile" "vga_module.kicad_sch"
+		(property "Sheetfile" "gfx_module.kicad_sch"
 			(at 190.5 166.9546 0)
 			(effects
@@
 			)
 		)
+		(pin "~{gfx_{ce}}" input
+			(at 190.5 157.48 180)
+			(effects
+				(font
+					(size 1.27 1.27)
+				)
+				(justify left)
+			)
+		)
+		(pin "data_{cpu}[0..7]" input
+			(at 190.5 134.62 180)
+			(effects
+				(font
+					(size 1.27 1.27)
+				)
+				(justify left)
+			)
+		)
+		(pin "clk_{2}" input
+			(at 190.5 125.73 180)
+			(effects
+				(font
+					(size 1.27 1.27)
+				)
+				(justify left)
+			)
+		)
+		(pin "~{we_{cpu}}" input
+			(at 190.5 161.29 180)
+			(effects
+				(font
+					(size 1.27 1.27)
+				)
+				(justify left)
+			)
+		)
+		(pin "~{ramb0_{ce}}" input
+			(at 190.5 153.67 180)
+			(effects
+				(font
+					(size 1.27 1.27)
+				)
+				(justify left)
+			)
+		)
+		(pin "~{oe_{cpu}}" input
+			(at 190.5 163.83 180)
+			(effects
+				(font
+					(size 1.27 1.27)
+				)
+				(justify left)
+			)
+		)
+		(pin "addr_{cpu}[0..15]" input
+			(at 190.5 130.81 180)
+			(effects
+				(font
+					(size 1.27 1.27)
+				)
+				(justify left)
+			)
+		)
+		(pin "~{plt_{cs}}" input
+			(at 190.5 149.86 180)
+			(effects
+				(font
+					(size 1.27 1.27)
+				)
+				(justify left)
+			)
+		)
+		(pin "gfx_{fr_start}" output
+			(at 237.744 133.35 0)
+			(effects
+				(font
+					(size 1.27 1.27)
+				)
+				(justify right)
+			)
+		)
+		(pin "gfx_{fr_prog}" output
+			(at 237.744 137.16 0)
+			(effects
+				(font
+					(size 1.27 1.27)
+				)
+				(justify right)
+			)
+		)
+		(pin "gfx_{dma_act}" output
+			(at 237.744 144.78 0)
+			(effects
+				(font
+					(size 1.27 1.27)
+				)
+				(justify right)
+			)
+		)
+		(pin "gfx_{fr_end}" output
+			(at 237.744 140.97 0)
+			(effects
+				(font
+					(size 1.27 1.27)
+				)
+				(justify right)
+			)
+		)

Commit message: update
Other:
- sheet gfx_module ports: added addr_{cpu}[0..12], clk, ram_{page}[0..1], ~{ce_{dma}}, ~{ce_{plt}}, ~{ce_{ram}}, ~{ce_{vga}}, ~{oe_{driver}}; removed addr_{cpu}[0..15], clk_{2}, ~{gfx_{ce}}, ~{plt_{cs}}, ~{ramb0_{ce}}
Changed lines of the file:
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@@
-			)
-		)
-		(pin "~{gfx_{ce}}" input
-			(at 190.5 157.48 180)
-			(effects
-				(font
-					(size 1.27 1.27)
-				)
-				(justify left)
 			)
 		)
 		(pin "data_{cpu}[0..7]" input
 			(at 190.5 134.62 180)
-			(effects
-				(font
-					(size 1.27 1.27)
-				)
-				(justify left)
-			)
-		)
-		(pin "clk_{2}" input
-			(at 190.5 125.73 180)
 			(effects
 				(font
@@
 			)
 		)
-		(pin "~{ramb0_{ce}}" input
-			(at 190.5 153.67 180)
-			(effects
-				(font
-					(size 1.27 1.27)
-				)
-				(justify left)
-			)
-		)
 		(pin "~{oe_{cpu}}" input
 			(at 190.5 163.83 180)
-			(effects
-				(font
-					(size 1.27 1.27)
-				)
-				(justify left)
-			)
-		)
-		(pin "addr_{cpu}[0..15]" input
-			(at 190.5 130.81 180)
-			(effects
-				(font
-					(size 1.27 1.27)
-				)
-				(justify left)
-			)
-		)
-		(pin "~{plt_{cs}}" input
-			(at 190.5 149.86 180)
 			(effects
 				(font
@@
 			(effects
 				(font
+					(size 1.27 1.27)
+				)
+				(justify right)
+			)
+		)
+		(pin "~{oe_{driver}}" input
+			(at 190.5 139.7 180)
+			(effects
+				(font
+					(size 1.27 1.27)
+				)
+				(justify left)
+			)
+		)
+		(pin "clk" input
+			(at 190.5 143.51 180)
+			(effects
+				(font
+					(size 1.27 1.27)
+				)
+				(justify left)
+			)
+		)
+		(pin "~{ce_{ram}}" input
+			(at 190.5 147.32 180)
+			(effects
+				(font
+					(size 1.27 1.27)
+				)
+				(justify left)
+			)
+		)
+		(pin "~{ce_{dma}}" input
+			(at 190.5 152.4 180)
+			(effects
+				(font
+					(size 1.27 1.27)
+				)
+				(justify left)
+			)
+		)
+		(pin "addr_{cpu}[0..12]" input
+			(at 190.5 156.21 180)
+			(effects
+				(font
+					(size 1.27 1.27)
+				)
+				(justify left)
+			)
+		)
+		(pin "ram_{page}[0..1]" input
+			(at 190.5 127 180)
+			(effects
+				(font
+					(size 1.27 1.27)
+				)
+				(justify left)
+			)
+		)
+		(pin "~{ce_{plt}}" input
+			(at 190.5 130.81 180)
+			(effects
+				(font
+					(size 1.27 1.27)
+				)
+				(justify left)
+			)
+		)
+		(pin "~{ce_{vga}}" input
+			(at 208.28 122.174 90)
+			(effects
+				(font
