File: hardware/kicad/dd8_computer/gfx_module.kicad_sch (KiCad schematic)
At the start: 26 parts, among them J1 VGA_CONN, U1 VGA, U14 SN74ACT244, U15 SN74ACT244, U16 SN74ACT244, U17 SN74ACT244, U18 SN74ACT244, U19 AS7C256B, U2 DMA, U21 AS7C256B, U22 AS7C256B, U24 LA35PDG, U25 SN74HC574N, U26 SN74HC574N

Commit message: updates
Parts:
- removed D5, D6, D7, D8: BAT85, symbol Device:D_Schottky
- removed R10, R9: R, symbol Device:R
- removed R15, R16: R_Small, symbol Device:R_Small
- removed U17, U18: SN74ACT244, symbol dd8_components_library:SN74ACT244
- added R1, R2, R3: R, symbol Device:R
- added U3: SN74AC245N, symbol dd8_components_library:SN74AC245N
Connections:
- net addr_{cpu}13 is gone; now on net ram_{bank}1: U15. (~{2OE})
- net addr_{cpu}14 is gone; now on net ram_{bank}1: U15. (~{2OE})
- net va15 is gone; now on net ~{vram0_{ce}}: U21.20 (~{CE})
- net ~{va15} is gone; now on net ~{vram1_{ce}}: U22.20 (~{CE})
- net GND: now also U3. (~{OE})
- net VCC: now also R1.2, R2.2, R3.2, U3. (~{OE})
- net data_{cpu}0: now also U3. (~{OE})
- net data_{cpu}1: now also U3. (~{OE})
- net data_{cpu}2: now also U3. (~{OE})
- net data_{cpu}3: now also U3. (~{OE})
- net data_{cpu}4: now also U3. (~{OE})
- net data_{cpu}5: now also U3. (~{OE})
- net data_{cpu}6: now also U3. (~{OE})
- net data_{cpu}7: now also U3. (~{OE})
- net gfx_{dma_act}: now also R1.1, U3. (~{OE})
- net rd0: now also U3. (~{OE})
- net rd1: now also U3. (~{OE})
- net rd2: now also U3. (~{OE})
- net rd3: now also U3. (~{OE})
- net rd4: now also U3. (~{OE})
- net rd5: now also U3. (~{OE})
- net rd6: now also U3. (~{OE})
- net rd7: now also U3. (~{OE})
- net ~{oe_{cpu}}: now also U3. (~{OE})
- net ~{vram0_{ce}}: now also R2.1
- net ~{vram1_{ce}}: now also R3.1
- net ram_{bank}1: now reaches U15. (~{2OE})
- new net ram_{bank}0: U15. (~{2OE})
- no-connect marks 0 -> 20
Other:
- note added: "do we need this ?"

Commit message: updates
Parts:
- removed R1, R11, R12, R13, R14, R2, R3: R, symbol Device:R
- added U4, U5: ~, symbol dd8_components_library:dd8_addr_mux
Connections:
- net ram_{bank}0 is gone; now on net ram_{page}1: U15. (~{2OE})
- net ram_{bank}1 is gone; now on net ram_{page}1: U15. (~{2OE})
- net ~{ramb0_{ce}} is gone; now on net ~{we_{cpu}}: U16. (~{2OE})
- net GND: now also U1. (~{VGA_OUT}), U2. (~{S_{WE}}), U4. (~{YA_{7}}), U5. (~{YA_{7}})
- net addr_{cpu}0: now also U1. (~{VGA_OUT})
- net addr_{cpu}1: now also U1. (~{VGA_OUT})
- net clk_{2}: no longer U16. (~{2OE}), U2. (~{S_{WE}})
- net data_{cpu}0: now also U1. (~{VGA_OUT})
- net data_{cpu}1: now also U1. (~{VGA_OUT})
- net data_{cpu}2: now also U1. (~{VGA_OUT})
- net data_{cpu}3: now also U1. (~{VGA_OUT})
- net data_{cpu}4: now also U1. (~{VGA_OUT})
- net data_{cpu}5: now also U1. (~{VGA_OUT})
- net data_{cpu}6: now also U1. (~{VGA_OUT})
- net data_{cpu}7: now also U1. (~{VGA_OUT})
- net gfx_{dma_act}: no longer U14. (~{2OE}), U15. (~{2OE}), U16. (~{2OE}), U2. (~{S_{WE}}), U3. (~{OE})
- net gfx_{fr_end}: no longer U1. (~{VGA_OUT})
- net gfx_{fr_prog}: no longer U1. (~{VGA_OUT})
- net gfx_{fr_start}: no longer U1. (~{VGA_OUT})
- net ~{oe_{cpu}}: no longer U3. (~{OE})
- net ~{ram_{ce}}: no longer U19.20 (~{CE})
- net ~{vga_{ce}}: now also U1. (~{VGA_OUT})
- net ram_{page}1: now reaches U15. (~{2OE})
- net VCC renamed +5V
- net +5V: now also U1. (~{VGA_OUT}), U2. (~{S_{WE}}), U4. (~{YA_{7}}), U5. (~{YA_{7}})
- removed net clk_{gfx}: U1. (~{VGA_OUT}), U16. (~{2OE}), U2. (~{S_{WE}})
- net h_sync: no longer names the net of U26.2 (1D)
- net h_sync: no longer U1. (~{VGA_OUT})
- net pd0 renamed pix_{data}0
- net pd1 renamed pix_{data}1
- net pd2 renamed pix_{data}2
- net pd3 renamed pix_{data}3
- net pd4 renamed pix_{data}4
- net pd5 renamed pix_{data}5
- net pd6 renamed pix_{data}6
- net pd7 renamed pix_{data}7
- net pd8 renamed pix_{data}8
- net pd9 renamed pix_{data}9
- removed net ra0: U1. (~{VGA_OUT}), U14. (~{2OE}), U19.10 (A0), U2. (~{S_{WE}})
- removed net ra1: U1. (~{VGA_OUT}), U14. (~{2OE}), U19.9 (A1), U2. (~{S_{WE}})
- removed net ra10: U15. (~{2OE}), U19.21 (A10), U2. (~{S_{WE}})
- removed net ra11: U15. (~{2OE}), U19.23 (A11), U2. (~{S_{WE}})
- removed net ra12: U15. (~{2OE}), U19.2 (A12), U2. (~{S_{WE}})
- removed net ra13: U15. (~{2OE}), U19.26 (A13), U2. (~{S_{WE}})
- removed net ra14: U15. (~{2OE}), U19.1 (A14), U2. (~{S_{WE}})
- removed net ra2: U14. (~{2OE}), U19.8 (A2), U2. (~{S_{WE}})
- removed net ra3: U1. (~{VGA_OUT}), U14. (~{2OE}), U19.7 (A3), U2. (~{S_{WE}})
- removed net ra4: U14. (~{2OE}), U19.6 (A4), U2. (~{S_{WE}})
- removed net ra5: U14. (~{2OE}), U19.5 (A5), U2. (~{S_{WE}})
- removed net ra6: U14. (~{2OE}), U19.4 (A6), U2. (~{S_{WE}})
- removed net ra7: U14. (~{2OE}), U19.3 (A7), U2. (~{S_{WE}})
- removed net ra8: U15. (~{2OE}), U19.25 (A8), U2. (~{S_{WE}})
- removed net ra9: U15. (~{2OE}), U19.24 (A9), U2. (~{S_{WE}})
- removed net rd0: U1. (~{VGA_OUT}), U19.11 (DQ0), U2. (~{S_{WE}}), U3. (~{OE})
- removed net rd1: U1. (~{VGA_OUT}), U19.12 (DQ1), U2. (~{S_{WE}}), U3. (~{OE})
- removed net rd2: U1. (~{VGA_OUT}), U19.13 (DQ2), U2. (~{S_{WE}}), U3. (~{OE})
- removed net rd3: U1. (~{VGA_OUT}), U19.15 (DQ3), U2. (~{S_{WE}}), U3. (~{OE})
- removed net rd4: U1. (~{VGA_OUT}), U19.16 (DQ4), U2. (~{S_{WE}}), U3. (~{OE})
- removed net rd5: U1. (~{VGA_OUT}), U19.17 (DQ5), U2. (~{S_{WE}}), U3. (~{OE})
- removed net rd6: U1. (~{VGA_OUT}), U19.18 (DQ6), U2. (~{S_{WE}}), U3. (~{OE})
- removed net rd7: U1. (~{VGA_OUT}), U19.19 (DQ7), U2. (~{S_{WE}}), U3. (~{OE})
- net rgb0 renamed data_{rgb}0
- net rgb1 renamed data_{rgb}1
- net rgb2 renamed data_{rgb}2
- net rgb3 renamed data_{rgb}3
- net rgb4 renamed data_{rgb}4
- net rgb5 renamed data_{rgb}5
- net rgb6 renamed data_{rgb}6
- net rgb7 renamed data_{rgb}7
- net v_sync: no longer names the net of U26.3 (2D)
- net v_sync: no longer U1. (~{VGA_OUT})
- net va0 renamed vaddr0
- net vaddr0: no longer U1. (~{VGA_OUT}), U2. (~{S_{WE}})
- net va1 renamed vaddr1
- net vaddr1: now also U4. (~{YA_{7}}); no longer U1. (~{VGA_OUT}), U2. (~{S_{WE}})
- net va10 renamed vaddr10
- net vaddr10: now also U5. (~{YA_{7}}); no longer U1. (~{VGA_OUT}), U2. (~{S_{WE}})
- net va11 renamed vaddr11
- net vaddr11: now also U5. (~{YA_{7}}); no longer U1. (~{VGA_OUT}), U2. (~{S_{WE}})
- net va12 renamed vaddr12
- net vaddr12: now also U5. (~{YA_{7}}); no longer U1. (~{VGA_OUT}), U2. (~{S_{WE}})
- net va13 renamed vaddr13
- net vaddr13: now also U5. (~{YA_{7}}); no longer U1. (~{VGA_OUT}), U2. (~{S_{WE}})
- net va14 renamed vaddr14
- net vaddr14: now also U5. (~{YA_{7}}); no longer U1. (~{VGA_OUT}), U2. (~{S_{WE}})
- net va2 renamed vaddr2
- net vaddr2: now also U4. (~{YA_{7}}); no longer U1. (~{VGA_OUT}), U2. (~{S_{WE}})
- net va3 renamed vaddr3
- net vaddr3: now also U4. (~{YA_{7}}); no longer U1. (~{VGA_OUT}), U2. (~{S_{WE}})
- net va4 renamed vaddr4
- net vaddr4: now also U4. (~{YA_{7}}); no longer U1. (~{VGA_OUT}), U2. (~{S_{WE}})
- net va5 renamed vaddr5
- net vaddr5: now also U4. (~{YA_{7}}); no longer U1. (~{VGA_OUT}), U2. (~{S_{WE}})
- net va6 renamed vaddr6
- net vaddr6: now also U4. (~{YA_{7}}); no longer U1. (~{VGA_OUT}), U2. (~{S_{WE}})
- net va7 renamed vaddr7
- net vaddr7: now also U4. (~{YA_{7}}); no longer U1. (~{VGA_OUT}), U2. (~{S_{WE}})
- net va8 renamed vaddr8
- net vaddr8: now also U5. (~{YA_{7}}); no longer U1. (~{VGA_OUT}), U2. (~{S_{WE}})
- net va9 renamed vaddr9
- net vaddr9: now also U5. (~{YA_{7}}); no longer U1. (~{VGA_OUT}), U2. (~{S_{WE}})
- net vd0 renamed vdata0
- net vd1 renamed vdata1
- net vd2 renamed vdata2
- net vd3 renamed vdata3
- net vd4 renamed vdata4
- net vd5 renamed vdata5
- net vd6 renamed vdata6
- net vd7 renamed vdata7
- net vga_conn_b1: no longer names the net of J1.18 (Pin_18)
- net vga_conn_b1: no longer U25.17 (3Q)
- net vga_conn_b2: no longer names the net of J1.16 (Pin_16)
- net vga_conn_b2: no longer U25.14 (6Q)
- net vga_conn_g0: no longer names the net of J1.13 (Pin_13)
- net vga_conn_g0: no longer U25.18 (2Q)
- net vga_conn_g1: no longer names the net of J1.14 (Pin_14)
- net vga_conn_g1: no longer U25.15 (5Q)
- net vga_conn_g2: no longer names the net of J1.11 (Pin_11)
- net vga_conn_g2: no longer U25.12 (8Q)
- net vga_conn_h: no longer names the net of J1.7 (Pin_7)
- net vga_conn_h: no longer U26.19 (1Q)
- net vga_conn_r0: no longer names the net of J1.19 (Pin_19)
- net vga_conn_r0: no longer U25.19 (1Q)
- net vga_conn_r1: no longer names the net of J1.17 (Pin_17)
- net vga_conn_r1: no longer U25.16 (4Q)
- net vga_conn_r2: no longer names the net of J1.15 (Pin_15)
- net vga_conn_r2: no longer U25.13 (7Q)
- net vga_conn_v: no longer names the net of J1.8 (Pin_8)
- net vga_conn_v: no longer U26.18 (2Q)
- removed net vga_latch: U1. (~{VGA_OUT}), U25.11 (CLK), U26.11 (CLK)
- removed net ~{free_vbus}: U1. (~{VGA_OUT}), U2. (~{S_{WE}})
- removed net ~{gfx_{ce}}: U1. (~{VGA_OUT}), U16. (~{2OE}), U2. (~{S_{WE}})
- removed net ~{ram_{oe}}: U16. (~{2OE}), U19.22 (~{OE}), U2. (~{S_{WE}})
- removed net ~{ram_{we}}: U1. (~{VGA_OUT}), U16. (~{2OE}), U19.27 (~{WE}), U2. (~{S_{WE}})
- removed net ~{vga_active}: U1. (~{VGA_OUT}), U21.22 (~{OE}), U22.22 (~{OE})
- net ~{vga_enabled}: no longer names the net of U24.43 (~{OE}_{R}), U24.47 (~{CE}_{R})
- net ~{vga_enabled}: no longer U1. (~{VGA_OUT}), U26.1 (~{OE})
- net ~{vga_out}: no longer names the net of U25.1 (~{OE})
- net ~{vga_out}: no longer U1. (~{VGA_OUT})
- removed net ~{vram0_{ce}}: U1. (~{VGA_OUT}), U2. (~{S_{WE}}), U21.20 (~{CE})
- removed net ~{vram1_{ce}}: U1. (~{VGA_OUT}), U2. (~{S_{WE}}), U22.20 (~{CE})
- removed net ~{vram_{we}}: U2. (~{S_{WE}}), U21.27 (~{WE}), U22.27 (~{WE})
- new net addr_{dma}0: U14. (~{2OE}), U19.10 (A0), U2. (~{S_{WE}})
- new net addr_{dma}1: U14. (~{2OE}), U19.9 (A1), U2. (~{S_{WE}})
- new net addr_{dma}10: U15. (~{2OE}), U19.21 (A10), U2. (~{S_{WE}})
- new net addr_{dma}11: U15. (~{2OE}), U19.23 (A11), U2. (~{S_{WE}})
- new net addr_{dma}12: U15. (~{2OE}), U19.2 (A12), U2. (~{S_{WE}})
- new net addr_{dma}13: U15. (~{2OE}), U19.26 (A13), U2. (~{S_{WE}})
- new net addr_{dma}14: U15. (~{2OE}), U19.1 (A14), U2. (~{S_{WE}})
- new net addr_{dma}2: U14. (~{2OE}), U19.8 (A2), U2. (~{S_{WE}})
- new net addr_{dma}3: U14. (~{2OE}), U19.7 (A3), U2. (~{S_{WE}})
- new net addr_{dma}4: U14. (~{2OE}), U19.6 (A4), U2. (~{S_{WE}})
- new net addr_{dma}5: U14. (~{2OE}), U19.5 (A5), U2. (~{S_{WE}})
- new net addr_{dma}6: U14. (~{2OE}), U19.4 (A6), U2. (~{S_{WE}})
- new net addr_{dma}7: U14. (~{2OE}), U19.3 (A7), U2. (~{S_{WE}})
- new net addr_{dma}8: U15. (~{2OE}), U19.25 (A8), U2. (~{S_{WE}})
- new net addr_{dma}9: U15. (~{2OE}), U19.24 (A9), U2. (~{S_{WE}})
- new net data_{dma}0: U19.11 (DQ0), U2. (~{S_{WE}}), U3. (~{OE})
- new net data_{dma}1: U19.12 (DQ1), U2. (~{S_{WE}}), U3. (~{OE})
- new net data_{dma}2: U19.13 (DQ2), U2. (~{S_{WE}}), U3. (~{OE})
- new net data_{dma}3: U19.15 (DQ3), U2. (~{S_{WE}}), U3. (~{OE})
- new net data_{dma}4: U19.16 (DQ4), U2. (~{S_{WE}}), U3. (~{OE})
- new net data_{dma}5: U19.17 (DQ5), U2. (~{S_{WE}}), U3. (~{OE})
- new net data_{dma}6: U19.18 (DQ6), U2. (~{S_{WE}}), U3. (~{OE})
- new net data_{dma}7: U19.19 (DQ7), U2. (~{S_{WE}}), U3. (~{OE})
- new net dma_{active}: U14. (~{2OE}), U15. (~{2OE}), U16. (~{2OE}), U2. (~{S_{WE}}), U3. (~{OE})
- new net ram_{page}0: U15. (~{2OE})
- new net vaddr_{dma}0: U2. (~{S_{WE}}), U4. (~{YA_{7}})
- new net vaddr_{dma}1: U2. (~{S_{WE}}), U4. (~{YA_{7}})
- new net vaddr_{dma}10: U2. (~{S_{WE}}), U5. (~{YA_{7}})
- new net vaddr_{dma}11: U2. (~{S_{WE}}), U5. (~{YA_{7}})
- new net vaddr_{dma}12: U2. (~{S_{WE}}), U5. (~{YA_{7}})
- new net vaddr_{dma}13: U2. (~{S_{WE}}), U5. (~{YA_{7}})
- new net vaddr_{dma}14: U2. (~{S_{WE}}), U5. (~{YA_{7}})
- new net vaddr_{dma}15: U2. (~{S_{WE}}), U5. (~{YA_{7}})
- new net vaddr_{dma}2: U2. (~{S_{WE}}), U4. (~{YA_{7}})
- new net vaddr_{dma}3: U2. (~{S_{WE}}), U4. (~{YA_{7}})
- new net vaddr_{dma}4: U2. (~{S_{WE}}), U4. (~{YA_{7}})
- new net vaddr_{dma}5: U2. (~{S_{WE}}), U4. (~{YA_{7}})
- new net vaddr_{dma}6: U2. (~{S_{WE}}), U4. (~{YA_{7}})
- new net vaddr_{dma}7: U2. (~{S_{WE}}), U4. (~{YA_{7}})
- new net vaddr_{dma}8: U2. (~{S_{WE}}), U5. (~{YA_{7}})
- new net vaddr_{dma}9: U2. (~{S_{WE}}), U5. (~{YA_{7}})
- new net vaddr_{vga}0: U1. (~{VGA_OUT}), U4. (~{YA_{7}})
- new net vaddr_{vga}1: U1. (~{VGA_OUT}), U4. (~{YA_{7}})
- new net vaddr_{vga}10: U1. (~{VGA_OUT}), U5. (~{YA_{7}})
- new net vaddr_{vga}11: U1. (~{VGA_OUT}), U5. (~{YA_{7}})
- new net vaddr_{vga}12: U1. (~{VGA_OUT}), U5. (~{YA_{7}})
- new net vaddr_{vga}13: U1. (~{VGA_OUT}), U5. (~{YA_{7}})
- new net vaddr_{vga}14: U1. (~{VGA_OUT}), U5. (~{YA_{7}})
- new net vaddr_{vga}15: U1. (~{VGA_OUT}), U5. (~{YA_{7}})
- new net vaddr_{vga}2: U1. (~{VGA_OUT}), U4. (~{YA_{7}})
- new net vaddr_{vga}3: U1. (~{VGA_OUT}), U4. (~{YA_{7}})
- new net vaddr_{vga}4: U1. (~{VGA_OUT}), U4. (~{YA_{7}})
- new net vaddr_{vga}5: U1. (~{VGA_OUT}), U4. (~{YA_{7}})
- new net vaddr_{vga}6: U1. (~{VGA_OUT}), U4. (~{YA_{7}})
- new net vaddr_{vga}7: U1. (~{VGA_OUT}), U4. (~{YA_{7}})
- new net vaddr_{vga}8: U1. (~{VGA_OUT}), U5. (~{YA_{7}})
- new net vaddr_{vga}9: U1. (~{VGA_OUT}), U5. (~{YA_{7}})
- new net ~{dma_{ce}}: U16. (~{2OE})
- no-connect marks 20 -> 21
Other:
- note removed: "ADDRESS BUSS DRIVERS"
- note removed: "CONTROL SIGNAL DRIVER"
- note removed: "CPU RAM"
- note removed: "DATA BUSS DRIVERS"
- note removed: "DMA"
- note removed: "LATCH"
- note removed: "PALETTE DP RAM"
- note removed: "TODO: bypass caps, coupling caps, resistance conrete values"
- note removed: "VGA GEN."
- note removed: "VIDEO RAM"
- note removed: "clk_{gfx} shifted clk_{2}+10ns"
- note removed: "do we need this ?"
- moved on the sheet: J1, U14, U15, U16, U19, U21, U22, U24, U25, U26, U3

Commit message: update
Parts:
- added C1, C10, C11, C12, C13, C14, C15, C16, C17, C18, C19, C2, C20, C21, C22, C23, C24, C25, C26, C27, C28, C29, C3, C30, C31, C32, C4, C5, C6, C7, C8, C9: 100n, symbol Device:C_Small
- added R1, R2, R3, R4: 10k, symbol Device:R_Small
Connections:
- net ~{dma_{ce}} is gone; now on net ~{we_{dma}}: U16. (~{2OE})
- net ~{ram_{ce}} is gone; now on net ~{we_{dma}}: U16. (~{2OE})
- net ~{vga_{ce}} is gone; now on net ~{we_{cpu}}: U1. (~{VGA_OUT})
- net +5V: now also C1.1, C10.1, C11.1, C12.1, C13.1, C14.1, C15.1, C16.1, C17.1, C18.1, C19.1, C2.1, C20.1, C21.1, C22.1, C23.1, C24.1, C25.1, C26.1, C27.1, C28.1, C29.1, C3.1, C30.1, C31.1, C32.1, C4.1, C5.1, C6.1, C7.1, C8.1, C9.1, R1.1, R4.1
- net GND: now also C1.2, C10.2, C11.2, C12.2, C13.2, C14.2, C15.2, C16.2, C17.2, C18.2, C19.2, C2.2, C20.2, C21.2, C22.2, C23.2, C24.2, C25.2, C26.2, C27.2, C28.2, C29.2, C3.2, C30.2, C31.2, C32.2, C4.2, C5.2, C6.2, C7.2, C8.2, C9.2, R2.2, R3.2
- net dma_{active}: no longer U16. (~{2OE}), U2. (~{S_{WE}}), U3. (~{OE})
- net gfx_{dma_act}: now also U14. (~{2OE}), U15. (~{2OE}), U16. (~{2OE}), U2. (~{S_{WE}}), U3. (~{OE})
- net gfx_{fr_end}: now also U1. (~{VGA_OUT})
- net gfx_{fr_prog}: now also U1. (~{VGA_OUT})
- net gfx_{fr_start}: now also U1. (~{VGA_OUT})
- net vaddr0: now also U4. (~{YA_{7}})
- net ~{we_{dma}}: now reaches U2. (~{S_{WE}})
- net ~{we_{dma}}: now also U19.27 (~{WE}), R4.2
- net data_{g2}: now reaches J1.11 (Pin_11)
- net data_{g2}: now also U25.12 (8Q)
- net data_{g0}: now reaches J1.13 (Pin_13)
- net data_{g0}: now also U25.18 (2Q)
- net data_{g1}: now reaches J1.14 (Pin_14)
- net data_{g1}: now also U25.15 (5Q)
- net data_{r2}: now reaches J1.15 (Pin_15)
- net data_{r2}: now also U25.13 (7Q)
- net data_{b2}: now reaches J1.16 (Pin_16)
- net data_{b2}: now also U25.14 (6Q)
- net data_{r1}: now reaches J1.17 (Pin_17)
- net data_{r1}: now also U25.16 (4Q)
- net data_{b1}: now reaches J1.18 (Pin_18)
- net data_{b1}: now also U25.17 (3Q)
- net data_{r0}: now reaches J1.19 (Pin_19)
- net data_{r0}: now also U25.19 (1Q)
- net vga_{hsync}: now reaches J1.7 (Pin_7)
- net vga_{hsync}: now also U26.19 (1Q)
- net vga_{vsync}: now reaches J1.8 (Pin_8)
- net vga_{vsync}: now also U26.18 (2Q)
- net at U21.20 (~{CE}): now also U5. (~{YA_{7}})
- net dma_{dst_as}: now reaches U21.22 (~{OE})
- net dma_{dst_as}: now also U2. (~{S_{WE}}), U22.22 (~{OE}), U4. (~{YA_{7}}), U5. (~{YA_{7}})
- net ~{dma_{dst_we}}: now reaches U21.27 (~{WE})
- net ~{dma_{dst_we}}: now also U2. (~{S_{WE}}), U22.27 (~{WE})
- net at U24.43 (~{OE}_{R}), U24.47 (~{CE}_{R}): now also U1. (~{VGA_OUT}), U26.1 (~{OE})
- net at U25.1 (~{OE}): now also U1. (~{VGA_OUT})
- net at U25.11 (CLK): now also U1. (~{VGA_OUT}), U26.11 (CLK)
- net ~{ce_{ram}}: now reaches U19.20 (~{CE})
- net ~{ce_{ram}}: now also U16. (~{2OE}), R3.1
- net ~{oe_{dma}}: now reaches U19.22 (~{OE})
- net ~{oe_{dma}}: now also U16. (~{2OE}), R2.1
- net at U26.2 (1D): now also U1. (~{VGA_OUT})
- net at U26.3 (2D): now also U1. (~{VGA_OUT})
- net ~{oe_{driver}}: now reaches U3. (~{OE})
- net at U22.20 (~{CE}): now also U5. (~{YA_{7}})
- net ~{plt_{cs}} renamed ~{ce_{plt}}
- new net: U1. (~{VGA_OUT}), U2. (~{S_{WE}})
- new net clk: U16. (~{2OE}), U2. (~{S_{WE}})
- new net clk_{d5ns}: U1. (~{VGA_OUT}), U16. (~{2OE}), U2. (~{S_{WE}})
- new net ~{ce_{dma}}: R1.2, U16. (~{2OE}), U2. (~{S_{WE}})
- new net ~{ce_{vga}}: U1. (~{VGA_OUT})
- no-connect marks 21 -> 22
Other:
- note added: "ADDR MUX 0"
- note added: "ADDR MUX 1"
- note added: "ADDR, DATA, CTRL BUS DRIVERS"
- note added: "ADDR. MUX."
- note added: "BUS DRIVERS"
- note added: "COLOR PLT. RAM"
- note added: "DMA CONTROLLER"
- note added: "DMA CTRL"
- note added: "GP. RAM"
- note added: "LATCH"
- note added: "PLT. RAM"
- note added: "VGA CONTROLLER"
- note added: "VGA CTRL"
- note added: "VIDEO RAM"
- moved on the sheet: J1
